File: KiCAD/Attenuator Controller Board/Attenuator Controller Board.kicad_pcb (KiCad board)
At the start: 2 copper layers, 100 x 70 mm, 33 parts, among them J1 Barrel_Jack_Switch, J2 Conn_Coaxial, J3 Conn_Coaxial, J4 Conn_01x24_Female, J5 DSub_15_HD, J6 DSub9, J7 DSub9, J8 DSub9, J9 Conn_01x24_Female, U1 ADM3307EARUZ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

Commit message: Complete draft - all connected - need to double check pinouts
Parts:
- moved LOGO3 46.9 mm to (159.6, 126.8)
- moved LOGO1 34.5 mm to (168.8, 125.3)
- moved LOGO2 3.14 mm to (119.1, 108.0)
- moved J5 0.39 mm to (198.4, 105.5)
Connections:
- D1 pad 3: /Analog_Input2 -> /Analog_Input1
- D1 pad 6: /Analog_Input1 -> /Analog_Input2
- RN1 pad 1: /Analog_Input2 -> /Analog_Input1
- RN1 pad 2: /Analog_Input1 -> /Analog_Input2
- U3 pad 31: /Analog_Input1 -> /Analog_Input2
- U3 pad 32: /Analog_Input2 -> /Analog_Input1
Routing:
- net /Motor(-): track 20.9 -> 33.0 mm
- net GND: track 782.7 -> 788.8 mm, vias 228 -> 246
- net /Analog_Input1: track 31.4 -> 28.1 mm
- net /Analog_Input2: track 28.1 -> 30.7 mm
Other:
- board text added: "5V DC"
- board text added: "Analog/Digital Input 1"
- board text added: "Analog/Digital Input 2"
- board text added: "Attenuator Controller Board"
- board text added: "Motor"
- board text added: "Serial 1"
- board text added: "Serial 2"
- board text added: "Serial 3"
- board text added: "https://github.com/Llamero/Attenuator_Controller_Board Designed by: Benjamin E. Smith Funded in part by: NIH P30EY003176"

Commit message: Motor pinout now matches K-cube specification
https://www.thorlabs.com/newgrouppage9.cfm?objectgroup_id=2419
Parts:
- U3: value Teensy3.6 -> Teensy3.5
- moved D1 5.18 mm to (144.8, 91.1)
- moved U2 0.86 mm to (182.6, 104.5)
- moved C10 0.60 mm to (174.0, 101.4)
- moved C9 0.60 mm to (176.8, 101.4)
Connections:
- J5 pad 10: /Ident-Vcc -> Net-(C10-Pad1)
- J5 pad 11: /Encoder(B) -> /Encoder(A)
- J5 pad 13: /Encoder(A) -> /Encoder(B)
- J5 pad 2: Net-(J5-Pad2) -> /Forward_Limit_Switch
- J5 pad 3: /Limit_Switch -> /Reverse_Limit_Switch
- J5 pad 5: /Motor(+) -> /Motor(-)
- J5 pad 7: /Motor(-) -> /Motor(+)
- J5 pad 9: /Ident(-) -> /Ident_In
- RN1 pad 3: /Ident(-) -> GND
- RN1 pad 4: (no net) -> /Ident_In
- RN1 pad 5: (no net) -> /Ident(-)
- RN1 pad 6: GND -> /Ident(-)
- U2 pad 5: /Motor(-) -> /Motor(+)
- U2 pad 7: /Motor(+) -> /Motor(-)
- U3 pad 19: /Ident-Vcc -> /Reverse_Limit_Switch
- U3 pad 21: /Limit_Switch -> /Encoder(B)
- U3 pad 23: /Encoder(A) -> /Forward_Limit_Switch
- U3 pad 24: /Encoder(B) -> /Encoder(A)
- U3 pad 30: /Ident(-) -> /NC33
- U3 pad 31: /Analog_Input2 -> /NC34
- U3 pad 32: /Analog_Input1 -> /NC35
- U3 pad 33: /NC36 -> /Ident(-)
- U3 pad 36: /NC39 -> /Analog_Input2
- U3 pad 41: /NC14 -> /Analog_Input1
Routing:
- net /Ident_In: track 0.00 -> 84.8 mm
- net /Ident(-): track 93.4 -> 13.1 mm
- net /Ident-Vcc: track 59.4 -> 0.00 mm
- net /Reverse_Limit_Switch: track 0.00 -> 57.4 mm
- net /Limit_Switch: track 52.0 -> 0.00 mm
- net /Forward_Limit_Switch: track 0.00 -> 45.4 mm
- net /Analog_Input2: track 30.7 -> 10.5 mm
- net Net-(C10-Pad1): track 56.1 -> 74.5 mm
- net /Encoder(B): track 38.9 -> 53.7 mm
- net /Motor(+): track 18.2 -> 33.0 mm, vias 0 -> 6
- net /Motor(-): track 33.0 -> 19.0 mm, vias 6 -> 0
- net /Alarm1: track 40.2 -> 30.8 mm
- net /Encoder(A): track 45.2 -> 39.1 mm
- net /3v3: track 34.6 -> 40.1 mm
- net GND: track 788.8 -> 794.1 mm, vias 246 -> 261
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Other:
- board text added: "Motor Control"
- board text added: "Teensy 3.5"
- board text removed: "Motor"
