File: KiCAD/Attenuator Controller Board/Attenuator Controller Board.sch (KiCad schematic (older format))
At the start: 33 parts, among them J1 Barrel_Jack_Switch, J2 Conn_Coaxial, J3 Conn_Coaxial, J4 Conn_01x24_Female, J5 DSub_15_HD, J6 DSub9, J7 DSub9, J8 DSub9, J9 Conn_01x24_Female, U1 ADM3307EARUZ, U2 ZXMHC3A01T8TA, U3 Teensy3.6

Commit message: More DSub-15 connections
Parts:
- BZ1: symbol Custom_parts:CPT-2016-75-SMT-TR -> Attenuator-Controller-Board-rescue:CPT-2016-75-SMT-TR-Custom_parts
- D1: symbol Custom_parts:BAT54BRW -> Attenuator-Controller-Board-rescue:BAT54BRW-Custom_parts
Connections:
- net labels added: Ident-Vcc
- net labels removed: NC25
Changed lines of the file:
@@
 Text Label 12300 6500 2    50   ~ 0
 Motor(+)
-Text Label 12300 7000 2    50   ~ 0
-3v3
 Wire Wire Line
 	12300 6900 11900 6900
@@
 	13800 3000 14550 3000
 $Comp
-L Custom_parts:BAT54BRW D1
+L Attenuator-Controller-Board-rescue:BAT54BRW-Custom_parts D1
 U 1 1 5F7E5C45
 P 8850 5300
@@
 Audible alarm
 $Comp
-L Custom_parts:CPT-2016-75-SMT-TR BZ1
+L Attenuator-Controller-Board-rescue:CPT-2016-75-SMT-TR-Custom_parts BZ1
 U 1 1 5FE01F50
 P 14450 6900
@@
 Text Label 8600 3700 2    50   ~ 0
 Analog_Input1
-Text Label 11500 2500 2    50   ~ 0
+Text Label 11500 3500 2    50   ~ 0
 Alarm1
-Text Label 11500 2600 2    50   ~ 0
+Text Label 11500 3600 2    50   ~ 0
 Alarm2
 $Comp
@@
 Text Label 11500 2800 2    50   ~ 0
 NC24
-Text Label 11500 2900 2    50   ~ 0
-NC25
 Text Label 11500 3200 2    50   ~ 0
 NC28
@@
 	8000 8500 7900 8500
 Connection ~ 8000 8500
+Text Label 11500 2900 2    50   ~ 0
+Ident-Vcc
+Text Label 12300 7000 2    50   ~ 0
+Ident-Vcc
 $EndSCHEMATC

Commit message: DSub 9 aligned
Parts:
- J4, J9: symbol Attenuator-Controller-Board-rescue:Conn_01x24_Female-Custom_parts -> Attenuator-Controller-Board-rescue:Conn_01x24_Female-Custom_parts-Attenuator-Controller-Board-rescue
- J5: symbol Attenuator-Controller-Board-rescue:DSub_15_HD_-_200-015-263R001-Custom_parts -> Attenuator-Controller-Board-rescue:DSub_15_HD_-_200-015-263R001-Custom_parts-Attenuator-Controller-Board-rescue
- J6, J7, J8: symbol Attenuator-Controller-Board-rescue:K202XHT-E9P-N-Custom_parts -> Attenuator-Controller-Board-rescue:K202XHT-E9P-N-Custom_parts-Attenuator-Controller-Board-rescue
- U1: symbol Attenuator-Controller-Board-rescue:ADM3307EARU-REEL7-Custom_parts -> Attenuator-Controller-Board-rescue:ADM3307EARU-REEL7-Custom_parts-Attenuator-Controller-Board-rescue
- U2: symbol Attenuator-Controller-Board-rescue:ZXMHC3A01T8TA-Custom_parts -> Attenuator-Controller-Board-rescue:ZXMHC3A01T8TA-Custom_parts-Attenuator-Controller-Board-rescue
- U3: symbol Attenuator-Controller-Board-rescue:Teensy3.6-Custom_parts -> Attenuator-Controller-Board-rescue:Teensy3.6-Custom_parts-Attenuator-Controller-Board-rescue
Connections:
- net labels added: NC11, NC12, NC25, NC3v3, NC4
- net labels removed: NC27, NC28
Changed lines of the file:
@@
 $EndComp
 $Comp
-L Attenuator-Controller-Board-rescue:Teensy3.6-Custom_parts U3
+L Attenuator-Controller-Board-rescue:Teensy3.6-Custom_parts-Attenuator-Controller-Board-rescue U3
 U 1 1 61E48BF3
 P 12650 3450
@@
 	13800 1300 14550 1300
 $Comp
-L Attenuator-Controller-Board-rescue:Conn_01x24_Female-Custom_parts J9
+L Attenuator-Controller-Board-rescue:Conn_01x24_Female-Custom_parts-Attenuator-Controller-Board-rescue J9
 U 1 1 61E48BF4
 P 14750 2400
@@
 	11500 2700 10750 2700
 $Comp
-L Attenuator-Controller-Board-rescue:Conn_01x24_Female-Custom_parts J4
+L Attenuator-Controller-Board-rescue:Conn_01x24_Female-Custom_parts-Attenuator-Controller-Board-rescue J4
 U 1 1 61E48BF8
 P 10550 2400
@@
 $EndComp
 $Comp
-L Attenuator-Controller-Board-rescue:DSub_15_HD_-_200-015-263R001-Custom_parts J5
+L Attenuator-Controller-Board-rescue:DSub_15_HD_-_200-015-263R001-Custom_parts-Attenuator-Controller-Board-rescue J5
 U 1 1 61DCB380
 P 12300 6100
@@
 RS-232_RXD1
 Text Label 13850 1500 0    50   ~ 0
-3v3
+NC3v3
 Text Label 11500 3000 2    50   ~ 0
 Serial1-TX
 $Comp
-L Attenuator-Controller-Board-rescue:K202XHT-E9P-N-Custom_parts J6
+L Attenuator-Controller-Board-rescue:K202XHT-E9P-N-Custom_parts-Attenuator-Controller-Board-rescue J6
 U 1 1 61DE6B05
 P 12300 8050
@@
 $EndComp
 $Comp
-L Attenuator-Controller-Board-rescue:K202XHT-E9P-N-Custom_parts J7
+L Attenuator-Controller-Board-rescue:K202XHT-E9P-N-Custom_parts-Attenuator-Controller-Board-rescue J7
 U 1 1 61E2A63C
 P 13500 8050
@@
 Serial2-RX
 $Comp
-L Attenuator-Controller-Board-rescue:ZXMHC3A01T8TA-Custom_parts U2
+L Attenuator-Controller-Board-rescue:ZXMHC3A01T8TA-Custom_parts-Attenuator-Controller-Board-rescue U2
 U 1 1 61E4F5F5
 P 8450 6500
@@
 	8350 6750 8350 6850
 $Comp
-L Attenuator-Controller-Board-rescue:ADM3307EARU-REEL7-Custom_parts U1
+L Attenuator-Controller-Board-rescue:ADM3307EARU-REEL7-Custom_parts-Attenuator-Controller-Board-rescue U1
 U 1 1 61E61C14
 P 8400 8000
@@
 $EndComp
 $Comp
-L Attenuator-Controller-Board-rescue:K202XHT-E9P-N-Custom_parts J8
+L Attenuator-Controller-Board-rescue:K202XHT-E9P-N-Custom_parts-Attenuator-Controller-Board-rescue J8
 U 1 1 61DD8259
 P 14700 8050
@@
 Text Label 8400 8500 2    50   ~ 0
 Shutdown
-Text Label 11500 1800 2    50   ~ 0
+Text Label 11500 3300 2    50   ~ 0
 Limit_Switch
-Text Label 10050 1950 2    50   ~ 0
+Text Label 11500 3500 2    50   ~ 0
 Encoder(A)
-Text Label 9950 2050 2    50   ~ 0
+Text Label 11500 3600 2    50   ~ 0
 Encoder(B)
 Text Label 12300 6500 2    50   ~ 0
@@
 Text Label 8600 3700 2    50   ~ 0
 Analog_Input1
-Text Label 11500 3500 2    50   ~ 0
+Text Label 11500 3400 2    50   ~ 0
 Alarm1
-Text Label 11500 3600 2    50   ~ 0
+Text Label 11500 3200 2    50   ~ 0
 Alarm2
 $Comp
@@
 Text Label 11500 2800 2    50   ~ 0
 NC24
-Text Label 11500 3200 2    50   ~ 0
-NC28
 Text Label 13800 1600 0    50   ~ 0
 NC23
@@
 Text Label 11500 1400 2    50   ~ 0
 Serial1-RX
-Text Label 11500 3100 2    50   ~ 0
-NC27
 Text Label 11500 1500 2    50   ~ 0
 NC1
@@
 	8000 8500 7900 8500
 Connection ~ 8000 8500
-Text Label 11500 2900 2    50   ~ 0
+Text Label 11500 3100 2    50   ~ 0
 Ident-Vcc
 Text Label 12300 7000 2    50   ~ 0
 Ident-Vcc
+Text Label 11500 2900 2    50   ~ 0
+NC25
+Text Label 11500 2500 2    50   ~ 0
+NC11
+Text Label 11500 2600 2    50   ~ 0
+NC12
+Text Label 11500 1800 2    50   ~ 0
+NC4
 $EndSCHEMATC

Commit message: Complete draft - all connected - need to double check pinouts
Parts:
- BZ1: symbol Attenuator-Controller-Board-rescue:CPT-2016-75-SMT-TR-Custom_parts -> Attenuator-Controller-Board-rescue:CPT-2016-75-SMT-TR-Custom_parts-Attenuator-Controller-Board-rescue
- D1: symbol Attenuator-Controller-Board-rescue:BAT54BRW-Custom_parts -> Attenuator-Controller-Board-rescue:BAT54BRW-Custom_parts-Attenuator-Controller-Board-rescue
- J4, J9: symbol Attenuator-Controller-Board-rescue:Conn_01x24_Female-Custom_parts-Attenuator-Controller-Board-rescue -> Attenuator-Controller-Board-rescue:Conn_01x24_Female-Custom_parts-Attenuator-Controller-Board-rescue-Attenuator-Control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
- J5: symbol Attenuator-Controller-Board-rescue:DSub_15_HD_-_200-015-263R001-Custom_parts-Attenuator-Controller-Board-rescue -> Attenuator-Controller-Board-rescue:DSub_15_HD_-_200-015-263R001-Custom_parts-Attenuator-Controller-Board-rescue-Attenua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
- J6, J7, J8: symbol Attenuator-Controller-Board-rescue:K202XHT-E9P-N-Custom_parts-Attenuator-Controller-Board-rescue -> Attenuator-Controller-Board-rescue:K202XHT-E9P-N-Custom_parts-Attenuator-Controller-Board-rescue-Attenuator-Controller-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
- U1: symbol Attenuator-Controller-Board-rescue:ADM3307EARU-REEL7-Custom_parts-Attenuator-Controller-Board-rescue -> Attenuator-Controller-Board-rescue:ADM3307EARU-REEL7-Custom_parts-Attenuator-Controller-Board-rescue-Attenuator-Control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
- U2: symbol Attenuator-Controller-Board-rescue:ZXMHC3A01T8TA-Custom_parts-Attenuator-Controller-Board-rescue -> Attenuator-Controller-Board-rescue:ZXMHC3A01T8TA-Custom_parts-Attenuator-Controller-Board-rescue-Attenuator-Controller-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
- U3: symbol Attenuator-Controller-Board-rescue:Teensy3.6-Custom_parts-Attenuator-Controller-Board-rescue -> Attenuator-Controller-Board-rescue:Teensy3.6-Custom_parts-Attenuator-Controller-Board-rescue-Attenuator-Controller-Boar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
Changed lines of the file:
@@
 $EndComp
 $Comp
-L Attenuator-Controller-Board-rescue:Teensy3.6-Custom_parts-Attenuator-Controller-Board-rescue U3
+L Attenuator-Controller-Board-rescue:Teensy3.6-Custom_parts-Attenuator-Controller-Board-rescue-Attenuator-Controller-Board-rescue U3
 U 1 1 61E48BF3
 P 12650 3450
@@
 	13800 1300 14550 1300
 $Comp
-L Attenuator-Controller-Board-rescue:Conn_01x24_Female-Custom_parts-Attenuator-Controller-Board-rescue J9
+L Attenuator-Controller-Board-rescue:Conn_01x24_Female-Custom_parts-Attenuator-Controller-Board-rescue-Attenuator-Controller-Board-rescue J9
 U 1 1 61E48BF4
 P 14750 2400
@@
 	11500 2700 10750 2700
 $Comp
-L Attenuator-Controller-Board-rescue:Conn_01x24_Female-Custom_parts-Attenuator-Controller-Board-rescue J4
+L Attenuator-Controller-Board-rescue:Conn_01x24_Female-Custom_parts-Attenuator-Controller-Board-rescue-Attenuator-Controller-Board-rescue J4
 U 1 1 61E48BF8
 P 10550 2400
@@
 $EndComp
 $Comp
-L Attenuator-Controller-Board-rescue:DSub_15_HD_-_200-015-263R001-Custom_parts-Attenuator-Controller-Board-rescue J5
+L Attenuator-Controller-Board-rescue:DSub_15_HD_-_200-015-263R001-Custom_parts-Attenuator-Controller-Board-rescue-Attenuator-Controller-Board-rescue J5
 U 1 1 61DCB380
 P 12300 6100
@@
 Serial1-TX
 $Comp
-L Attenuator-Controller-Board-rescue:K202XHT-E9P-N-Custom_parts-Attenuator-Controller-Board-rescue J6
+L Attenuator-Controller-Board-rescue:K202XHT-E9P-N-Custom_parts-Attenuator-Controller-Board-rescue-Attenuator-Controller-Board-rescue J6
 U 1 1 61DE6B05
 P 12300 8050
@@
 $EndComp
 $Comp
-L Attenuator-Controller-Board-rescue:K202XHT-E9P-N-Custom_parts-Attenuator-Controller-Board-rescue J7
+L Attenuator-Controller-Board-rescue:K202XHT-E9P-N-Custom_parts-Attenuator-Controller-Board-rescue-Attenuator-Controller-Board-rescue J7
 U 1 1 61E2A63C
 P 13500 8050
@@
 Serial2-RX
 $Comp
-L Attenuator-Controller-Board-rescue:ZXMHC3A01T8TA-Custom_parts-Attenuator-Controller-Board-rescue U2
+L Attenuator-Controller-Board-rescue:ZXMHC3A01T8TA-Custom_parts-Attenuator-Controller-Board-rescue-Attenuator-Controller-Board-rescue U2
 U 1 1 61E4F5F5
 P 8450 6500
@@
 	8350 6750 8350 6850
 $Comp
-L Attenuator-Controller-Board-rescue:ADM3307EARU-REEL7-Custom_parts-Attenuator-Controller-Board-rescue U1
+L Attenuator-Controller-Board-rescue:ADM3307EARU-REEL7-Custom_parts-Attenuator-Controller-Board-rescue-Attenuator-Controller-Board-rescue U1
 U 1 1 61E61C14
 P 8400 8000
@@
 $EndComp
 $Comp
-L Attenuator-Controller-Board-rescue:K202XHT-E9P-N-Custom_parts-Attenuator-Controller-Board-rescue J8
+L Attenuator-Controller-Board-rescue:K202XHT-E9P-N-Custom_parts-Attenuator-Controller-Board-rescue-Attenuator-Controller-Board-rescue J8
 U 1 1 61DD8259
 P 14700 8050
@@
 	13800 3000 14550 3000
 $Comp
-L Attenuator-Controller-Board-rescue:BAT54BRW-Custom_parts D1
+L Attenuator-Controller-Board-rescue:BAT54BRW-Custom_parts-Attenuator-Controller-Board-rescue D1
 U 1 1 5F7E5C45
 P 8850 5300
@@
 Audible alarm
 $Comp
-L Attenuator-Controller-Board-rescue:CPT-2016-75-SMT-TR-Custom_parts BZ1
+L Attenuator-Controller-Board-rescue:CPT-2016-75-SMT-TR-Custom_parts-Attenuator-Controller-Board-rescue BZ1
 U 1 1 5FE01F50
 P 14450 6900
@@
 	0    1    1    0
 $EndComp
+Text Label 8650 5600 2    50   ~ 0
+Analog_Input1
 Text Label 9400 5200 0    50   ~ 0
+Analog_Input2
+Text Label 13800 3400 0    50   ~ 0
 Analog_Input1
-Text Label 8650 5600 2    50   ~ 0
-Analog_Input2
 Text Label 13800 3500 0    50   ~ 0
-Analog_Input1
-Text Label 13800 3400 0    50   ~ 0
 Analog_Input2
 $Comp
@@
 	1    0    0    -1
 $EndComp
-Text Label 8600 3700 2    50   ~ 0
+Text Label 8600 4250 2    50   ~ 0
 Analog_Input1
 Text Label 11500 3400 2    50   ~ 0
@@
 	1    0    0    -1
 $EndComp
-Text Label 8600 4250 2    50   ~ 0
+Text Label 8600 3700 2    50   ~ 0
 Analog_Input2
 $Comp

Commit message: Motor pinout now matches K-cube specification
https://www.thorlabs.com/newgrouppage9.cfm?objectgroup_id=2419
Parts:
- added unit 4 of RN1
- BZ1: symbol Attenuator-Controller-Board-rescue:CPT-2016-75-SMT-TR-Custom_parts-Attenuator-Controller-Board-rescue -> Attenuator-Controller-Board-rescue:CPT-2016-75-SMT-TR-Custom_parts-Attenuator-Controller-Board-rescue-Attenuator-Contro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
- D1: symbol Attenuator-Controller-Board-rescue:BAT54BRW-Custom_parts-Attenuator-Controller-Board-rescue -> Attenuator-Controller-Board-rescue:BAT54BRW-Custom_parts-Attenuator-Controller-Board-rescue-Attenuator-Controller-Board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
- U3: value Teensy3.6 -> Teensy3.5; Part # DEV-14058 -> DEV-14056
Connections:
- net labels added: Forward_Limit_Switch, Ident_In, NC33, NC34, NC35, Reverse_Limit_Switch
- net labels removed: Ident-Vcc, Limit_Switch, NC14, NC36, NC39
- wire segments 84 -> 87
- no-connect marks 63 -> 62
Other:
- note added: "Teensy 3.5 120 MHz Microcontroller"
- note removed: "Teensy 3.6 180 MHz Microcontroller"
- moved on the sheet: RN1C
Changed lines of the file:
@@
 P 12650 3450
 F 0 "U3" H 12650 5887 60  0000 C CNN
-F 1 "Teensy3.6" H 12650 5781 60  0000 C CNN
+F 1 "Teensy3.5" H 12650 5781 60  0000 C CNN
 F 2 "Custom Footprints:Teensy_3_6_with_headers" H 12650 3500 60  0001 C CNN
-F 3 "https://media.digikey.com/pdf/Data%20Sheets/Sparkfun%20PDFs/DEV-14058_Web.pdf" H 12650 5781 60  0001 C CNN
+F 3 "https://media.digikey.com/pdf/Data%20Sheets/Sparkfun%20PDFs/DEV-14056_Web.pdf" H 12650 5781 60  0001 C CNN
 F 4 "SparkFun Electronics" H 12650 3450 50  0001 C CNN "Manufacturer"
-F 5 "DEV-14058" H 12650 3450 50  0001 C CNN "Part #"
+F 5 "DEV-14056" H 12650 3450 50  0001 C CNN "Part #"
 	1    12650 3450
 	1    0    0    -1
@@
 	13800 3100 14550 3100
 Text Notes 11200 700  0    118  ~ 0
-Teensy 3.6 180 MHz Microcontroller
+Teensy 3.5 120 MHz Microcontroller
 $Comp
 L Graphic:Logo_Open_Hardware_Small LOGO1
@@
 	1    0    0    -1
 $EndComp
-NoConn ~ 12300 6200
 NoConn ~ 12300 6400
 NoConn ~ 12300 6600
@@
 $EndComp
 Text Label 12300 6300 2    50   ~ 0
-Limit_Switch
-Text Label 9600 6650 0    50   ~ 0
+Reverse_Limit_Switch
+Text Label 9600 6850 0    50   ~ 0
 Motor(+)
-Text Label 12300 6700 2    50   ~ 0
+Text Label 12300 6500 2    50   ~ 0
 Motor(-)
-Text Label 12300 6900 2    50   ~ 0
+Text Label 11600 6700 2    50   ~ 0
 Ident(-)
+Text Label 12300 7300 2    50   ~ 0
+Encoder(B)
 Text Label 12300 7100 2    50   ~ 0
-Encoder(B)
-Text Label 12300 7300 2    50   ~ 0
 Encoder(A)
 $Comp
@@
 	0    1    1    0
 $EndComp
-Text Label 9600 6850 0    50   ~ 0
+Text Label 9600 6650 0    50   ~ 0
 Motor(-)
 Text Label 10950 6750 0    50   ~ 0
@@
 Text Label 8400 8500 2    50   ~ 0
 Shutdown
+Text Label 11500 3600 2    50   ~ 0
+Encoder(A)
 Text Label 11500 3300 2    50   ~ 0
-Limit_Switch
-Text Label 11500 3500 2    50   ~ 0
-Encoder(A)
-Text Label 11500 3600 2    50   ~ 0
 Encoder(B)
-Text Label 12300 6500 2    50   ~ 0
+Text Label 12300 6700 2    50   ~ 0
 Motor(+)
 Wire Wire Line
@@
 L power:GND #PWR013
 U 1 1 61DFC087
-P 11600 6900
-F 0 "#PWR013" H 11600 6650 50  0001 C CNN
-F 1 "GND" V 11605 6772 50  0000 R CNN
-F 2 "" H 11600 6900 50  0001 C CNN
-F 3 "" H 11600 6900 50  0001 C CNN
-	1    11600 6900
-	0    1    1    0
-$EndComp
-Text Label 13800 3600 0    50   ~ 0
+P 11300 6900
+F 0 "#PWR013" H 11300 6650 50  0001 C CNN
+F 1 "GND" V 11305 6772 50  0000 R CNN
+F 2 "" H 11300 6900 50  0001 C CNN
+F 3 "" H 11300 6900 50  0001 C CNN
+	1    11300 6900
+	0    1    1    0
+$EndComp
+Text Label 13800 3300 0    50   ~ 0
 Ident(-)
 $Comp
@@
 	13800 3000 14550 3000
 $Comp
-L Attenuator-Controller-Board-rescue:BAT54BRW-Custom_parts-Attenuator-Controller-Board-rescue D1
+L Attenuator-Controller-Board-rescue:BAT54BRW-Custom_parts-Attenuator-Controller-Board-rescue-Attenuator-Controller-Board-rescue D1
 U 1 1 5F7E5C45
 P 8850 5300
@@
 Audible alarm
 $Comp
-L Attenuator-Controller-Board-rescue:CPT-2016-75-SMT-TR-Custom_parts-Attenuator-Controller-Board-rescue BZ1
+L Attenuator-Controller-Board-rescue:CPT-2016-75-SMT-TR-Custom_parts-Attenuator-Controller-Board-rescue-Attenuator-Controller-Board-rescue BZ1
 U 1 1 5FE01F50
 P 14450 6900
@@
 Text Label 9400 5200 0    50   ~ 0
 Analog_Input2
-Text Label 13800 3400 0    50   ~ 0
+Text Label 13800 2500 0    50   ~ 0
 Analog_Input1
-Text Label 13800 3500 0    50   ~ 0
+Text Label 13800 3000 0    50   ~ 0
 Analog_Input2
 $Comp
@@
 L Device:R_Pack04_Split RN1
 U 3 1 61FC5D93
-P 11750 6900
-F 0 "RN1" V 11650 6900 50  0000 C CNN
-F 1 "4.7k" V 11750 6900 50  0000 C CNN
-F 2 "Resistor_SMD:R_Array_Convex_4x1206" V 11670 6900 50  0001 C CNN
-F 3 "https://industrial.panasonic.com/cdbs/www-data/pdf/AOC0000/AOC0000C14.pdf" H 11750 6900 50  0001 C CNN
-F 4 "Panasonic Electronic Components" V 11750 6900 50  0001 C CNN "Manufacturer"
-F 5 "EXB-38V472JV" V 11750 6900 50  0001 C CNN "Part #"
-	3    11750 6900
-	0    -1   1    0
+P 11450 6900
+F 0 "RN1" V 11350 6900 50  0000 C CNN
+F 1 "4.7k" V 11450 6900 50  0000 C CNN
+F 2 "Resistor_SMD:R_Array_Convex_4x1206" V 11370 6900 50  0001 C CNN
+F 3 "https://industrial.panasonic.com/cdbs/www-data/pdf/AOC0000/AOC0000C14.pdf" H 11450 6900 50  0001 C CNN
+F 4 "Panasonic Electronic Components" V 11450 6900 50  0001 C CNN "Manufacturer"
+F 5 "EXB-38V472JV" V 11450 6900 50  0001 C CNN "Part #"
+	3    11450 6900
+	0    1    -1   0
 $EndComp
 $Comp
@@
 Text Label 13800 2400 0    50   ~ 0
 NC15
-Text Label 13800 2500 0    50   ~ 0
-NC14
 Text Label 13800 2600 0    50   ~ 0
 NC13
@@
 Text Label 13800 2900 0    50   ~ 0
 NC_DAC0
-Text Label 13800 3000 0    50   ~ 0
-NC39
 Text Label 13800 3100 0    50   ~ 0
 NC38
 Text Label 13800 3200 0    50   ~ 0
 NC37
-Text Label 13800 3300 0    50   ~ 0
-NC36
 $Comp
 L Device:C_Small C10
@@
 	8000 8500 7900 8500
 Connection ~ 8000 8500
-Text Label 11500 3100 2    50   ~ 0
-Ident-Vcc
-Text Label 12300 7000 2    50   ~ 0
-Ident-Vcc
 Text Label 11500 2900 2    50   ~ 0
 NC25
@@
 Text Label 11500 1800 2    50   ~ 0
 NC4
+Wire Wire Line
+	12300 7000 10650 7000
+Wire Wire Line
+	10650 7000 10650 6750
+Connection ~ 10650 6750
+Text Label 12300 6200 2    50   ~ 0
+Forward_Limit_Switch
+$Comp
+L Device:R_Pack04_Split RN1
+U 4 1 61E2DDA8
+P 11750 6900
+F 0 "RN1" V 11650 6900 50  0000 C CNN
+F 1 "4.7k" V 11750 6900 50  0000 C CNN
+F 2 "Resistor_SMD:R_Array_Convex_4x1206" V 11670 6900 50  0001 C CNN
+F 3 "https://industrial.panasonic.com/cdbs/www-data/pdf/AOC0000/AOC0000C14.pdf" H 11750 6900 50  0001 C CNN
+F 4 "Panasonic Electronic Components" V 11750 6900 50  0001 C CNN "Manufacturer"
+F 5 "EXB-38V472JV" V 11750 6900 50  0001 C CNN "Part #"
+	4    11750 6900
+	0    -1   1    0
+$EndComp
+Wire Wire Line
+	11600 6900 11600 6700
+Text Label 12300 6900 2    50   ~ 0
+Ident_In
+Text Label 11500 3100 2    50   ~ 0
+Reverse_Limit_Switch
+Text Label 11500 3500 2    50   ~ 0
+Forward_Limit_Switch
+Connection ~ 11600 6900
+Text Label 13800 3400 0    50   ~ 0
+NC35
+Text Label 13800 3500 0    50   ~ 0
+NC34
+Text Label 13800 3600 0    50   ~ 0
+NC33
 $EndSCHEMATC

Commit message: Re-order annotation - add 0.1µF bypass to bypass H-bridge
Parts:
- removed C1: 10µF, Custom Footprints:0508_Capacitor, symbol Device:C_Small
- added C11, C9: 0.1µF, Capacitor_SMD:C_0603_1608Metric, symbol Device:C_Small
- J4: renamed from J9; symbol Attenuator-Controller-Board-rescue:Conn_01x24_Female-Custom_parts-Attenuator-Controller-Board-rescue-Attenuator-Controller-Board-rescue -> Attenuator-Controller-Board-rescue:Conn_01x24_Female-Custom_parts-Attenuator-Controller-Board-rescue-Attenuator-Controller-Board-rescue-Attenuator-Controller-Board-rescue
- J5: renamed from J4; symbol Attenuator-Controller-Board-rescue:Conn_01x24_Female-Custom_parts-Attenuator-Controller-Board-rescue-Attenuator-Controller-Board-rescue -> Attenuator-Controller-Board-rescue:Conn_01x24_Female-Custom_parts-Attenuator-Controller-Board-rescue-Attenuator-Controller-Board-rescue-Attenuator-Controller-Board-rescue
- J6, J7, J8: symbol Attenuator-Controller-Board-rescue:K202XHT-E9P-N-Custom_parts-Attenuator-Controller-Board-rescue-Attenuator-Controller-Board-rescue -> Attenuator-Controller-Board-rescue:K202XHT-E9P-N-Custom_parts-Attenuator-Controller-Board-rescue-Attenuator-Controller-Board-rescue-Attenuator-Controller-Board-rescue
- J9: renamed from J5; symbol Attenuator-Controller-Board-rescue:DSub_15_HD_-_200-015-263R001-Custom_parts-Attenuator-Controller-Board-rescue-Attenuator-Controller-Board-rescue -> Attenuator-Controller-Board-rescue:DSub_15_HD_-_200-015-263R001-Custom_parts-Attenuator-Controller-Board-rescue-Attenuator-Controller-Board-rescue-Attenuator-Controller-Board-rescue
- U1: symbol Attenuator-Controller-Board-rescue:ADM3307EARU-REEL7-Custom_parts-Attenuator-Controller-Board-rescue-Attenuator-Controller-Board-rescue -> Attenuator-Controller-Board-rescue:ADM3307EARU-REEL7-Custom_parts-Attenuator-Controller-Board-rescue-Attenuator-Controller-Board-rescue-Attenuator-Controller-Board-rescue
- U2: symbol Attenuator-Controller-Board-rescue:ZXMHC3A01T8TA-Custom_parts-Attenuator-Controller-Board-rescue-Attenuator-Controller-Board-rescue -> Attenuator-Controller-Board-rescue:ZXMHC3A01T8TA-Custom_parts-Attenuator-Controller-Board-rescue-Attenuator-Controller-Board-rescue-Attenuator-Controller-Board-rescue
- U3: symbol Attenuator-Controller-Board-rescue:Teensy3.6-Custom_parts-Attenuator-Controller-Board-rescue-Attenuator-Controller-Board-rescue -> Attenuator-Controller-Board-rescue:Teensy3.6-Custom_parts-Attenuator-Controller-Board-rescue-Attenuator-Controller-Board-rescue-Attenuator-Controller-Board-rescue
- renumbered C2 to C1, C3 to C2, C4 to C3, C5 to C4, C6 to C5, C7 to C6, C8 to C7, C9 to C8, J3 to J2, J2 to J3
Connections:
- wire segments 87 -> 86
Other:
- moved on the sheet: C10, C8, J1, J2, J3, RN1A, RN1B
