File: KiCAD/Attenuator Controller Board/Attenuator Controller Board.sch (KiCad schematic (older format))
At the start: 34 parts, among them J1 Barrel_Jack_Switch, J2 Conn_Coaxial, J3 Conn_Coaxial, J4 Conn_01x24_Female, J5 Conn_01x24_Female, J6 DSub9, J7 DSub9, J8 DSub9, J9 DSub_15_HD, U1 ADM3307EARUZ, U2 ZXMHC3A01T8TA, U3 Teensy3.5

Commit message: Ground connector housing and standoffs
Parts:
- BZ1: symbol Attenuator-Controller-Board-rescue:CPT-2016-75-SMT-TR-Custom_parts-Attenuator-Controller-Board-rescue-Attenuator-Controller-Board-rescue -> Attenuator-Controller-Board-rescue:CPT-2016-75-SMT-TR-Custom_parts-Attenuator-Controller-Board-rescue-Attenuator-Controller-Board-rescue-Attenuator-Controller-Board-rescue
- D1: symbol Attenuator-Controller-Board-rescue:BAT54BRW-Custom_parts-Attenuator-Controller-Board-rescue-Attenuator-Controller-Board-rescue -> Attenuator-Controller-Board-rescue:BAT54BRW-Custom_parts-Attenuator-Controller-Board-rescue-Attenuator-Controller-Board-rescue-Attenuator-Controller-Board-rescue
- H1, H2, H3, H4: symbol Mechanical:MountingHole -> Mechanical:MountingHole_Pad
- J4, J5: symbol Attenuator-Controller-Board-rescue:Conn_01x24_Female-Custom_parts-Attenuator-Controller-Board-rescue-Attenuator-Controller-Board-rescue-Attenuator-Controller-Board-rescue -> Attenuator-Controller-Board-rescue:Conn_01x24_Female-Custom_parts-Attenuator-Controller-Board-rescue-Attenuator-Controller-Board-rescue-Attenuator-Controller-Board-rescue-Attenuator-Controller-Board-rescue
- J6, J7, J8: symbol Attenuator-Controller-Board-rescue:K202XHT-E9P-N-Custom_parts-Attenuator-Controller-Board-rescue-Attenuator-Controller-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 -> Custom_parts:K202XHT-E9P-N
- J9: symbol Attenuator-Controller-Board-rescue:DSub_15_HD_-_200-015-263R001-Custom_parts-Attenuator-Controller-Board-rescue-Attenua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 -> Custom_parts:DSub_15_HD_-_200-015-263R001
- U1: symbol Attenuator-Controller-Board-rescue:ADM3307EARU-REEL7-Custom_parts-Attenuator-Controller-Board-rescue-Attenuator-Controller-Board-rescue-Attenuator-Controller-Board-rescue -> Attenuator-Controller-Board-rescue:ADM3307EARU-REEL7-Custom_parts-Attenuator-Controller-Board-rescue-Attenuator-Controller-Board-rescue-Attenuator-Controller-Board-rescue-Attenuator-Controller-Board-rescue
- U2: symbol Attenuator-Controller-Board-rescue:ZXMHC3A01T8TA-Custom_parts-Attenuator-Controller-Board-rescue-Attenuator-Controller-Board-rescue-Attenuator-Controller-Board-rescue -> Attenuator-Controller-Board-rescue:ZXMHC3A01T8TA-Custom_parts-Attenuator-Controller-Board-rescue-Attenuator-Controller-Board-rescue-Attenuator-Controller-Board-rescue-Attenuator-Controller-Board-rescue
- U3: symbol Attenuator-Controller-Board-rescue:Teensy3.6-Custom_parts-Attenuator-Controller-Board-rescue-Attenuator-Controller-Board-rescue-Attenuator-Controller-Board-rescue -> Attenuator-Controller-Board-rescue:Teensy3.6-Custom_parts-Attenuator-Controller-Board-rescue-Attenuator-Controller-Board-rescue-Attenuator-Controller-Board-rescue-Attenuator-Controller-Board-rescue
Connections:
- wire segments 86 -> 89
Changed lines of the file:
@@
 $EndComp
 $Comp
-L Attenuator-Controller-Board-rescue:Teensy3.6-Custom_parts-Attenuator-Controller-Board-rescue-Attenuator-Controller-Board-rescue-Attenuator-Controller-Board-rescue U3
+L Attenuator-Controller-Board-rescue:Teensy3.6-Custom_parts-Attenuator-Controller-Board-rescue-Attenuator-Controller-Board-rescue-Attenuator-Controller-Board-rescue-Attenuator-Controller-Board-rescue U3
 U 1 1 61E48BF3
 P 12650 3450
@@
 	13800 1300 14550 1300
 $Comp
-L Attenuator-Controller-Board-rescue:Conn_01x24_Female-Custom_parts-Attenuator-Controller-Board-rescue-Attenuator-Controller-Board-rescue-Attenuator-Controller-Board-rescue J4
+L Attenuator-Controller-Board-rescue:Conn_01x24_Female-Custom_parts-Attenuator-Controller-Board-rescue-Attenuator-Controller-Board-rescue-Attenuator-Controller-Board-rescue-Attenuator-Controller-Board-rescue J4
 U 1 1 61E48BF4
 P 14750 2400
@@
 	11500 2700 10750 2700
 $Comp
-L Attenuator-Controller-Board-rescue:Conn_01x24_Female-Custom_parts-Attenuator-Controller-Board-rescue-Attenuator-Controller-Board-rescue-Attenuator-Controller-Board-rescue J5
+L Attenuator-Controller-Board-rescue:Conn_01x24_Female-Custom_parts-Attenuator-Controller-Board-rescue-Attenuator-Controller-Board-rescue-Attenuator-Controller-Board-rescue-Attenuator-Controller-Board-rescue J5
 U 1 1 61E48BF8
 P 10550 2400
@@
 $EndComp
 $Comp
-L Attenuator-Controller-Board-rescue:DSub_15_HD_-_200-015-263R001-Custom_parts-Attenuator-Controller-Board-rescue-Attenuator-Controller-Board-rescue-Attenuator-Controller-Board-rescue J9
+L Custom_parts:DSub_15_HD_-_200-015-263R001 J9
 U 1 1 61DCB380
 P 12300 6100
@@
 Serial1-TX
 $Comp
-L Attenuator-Controller-Board-rescue:K202XHT-E9P-N-Custom_parts-Attenuator-Controller-Board-rescue-Attenuator-Controller-Board-rescue-Attenuator-Controller-Board-rescue J6
+L Custom_parts:K202XHT-E9P-N J6
 U 1 1 61DE6B05
 P 12300 8050
@@
 $EndComp
 $Comp
-L Attenuator-Controller-Board-rescue:K202XHT-E9P-N-Custom_parts-Attenuator-Controller-Board-rescue-Attenuator-Controller-Board-rescue-Attenuator-Controller-Board-rescue J7
+L Custom_parts:K202XHT-E9P-N J7
 U 1 1 61E2A63C
 P 13500 8050
@@
 Serial2-RX
 $Comp
-L Attenuator-Controller-Board-rescue:ZXMHC3A01T8TA-Custom_parts-Attenuator-Controller-Board-rescue-Attenuator-Controller-Board-rescue-Attenuator-Controller-Board-rescue U2
+L Attenuator-Controller-Board-rescue:ZXMHC3A01T8TA-Custom_parts-Attenuator-Controller-Board-rescue-Attenuator-Controller-Board-rescue-Attenuator-Controller-Board-rescue-Attenuator-Controller-Board-rescue U2
 U 1 1 61E4F5F5
 P 8450 6500
@@
 	8350 6750 8350 6850
 $Comp
-L Attenuator-Controller-Board-rescue:ADM3307EARU-REEL7-Custom_parts-Attenuator-Controller-Board-rescue-Attenuator-Controller-Board-rescue-Attenuator-Controller-Board-rescue U1
+L Attenuator-Controller-Board-rescue:ADM3307EARU-REEL7-Custom_parts-Attenuator-Controller-Board-rescue-Attenuator-Controller-Board-rescue-Attenuator-Controller-Board-rescue-Attenuator-Controller-Board-rescue U1
 U 1 1 61E61C14
 P 8400 8000
@@
 $EndComp
 $Comp
-L Attenuator-Controller-Board-rescue:K202XHT-E9P-N-Custom_parts-Attenuator-Controller-Board-rescue-Attenuator-Controller-Board-rescue-Attenuator-Controller-Board-rescue J8
+L Custom_parts:K202XHT-E9P-N J8
 U 1 1 61DD8259
 P 14700 8050
@@
 	13800 3000 14550 3000
 $Comp
-L Attenuator-Controller-Board-rescue:BAT54BRW-Custom_parts-Attenuator-Controller-Board-rescue-Attenuator-Controller-Board-rescue D1
+L Attenuator-Controller-Board-rescue:BAT54BRW-Custom_parts-Attenuator-Controller-Board-rescue-Attenuator-Controller-Board-rescue-Attenuator-Controller-Board-rescue D1
 U 1 1 5F7E5C45
 P 8850 5300
@@
 Audible alarm
 $Comp
-L Attenuator-Controller-Board-rescue:CPT-2016-75-SMT-TR-Custom_parts-Attenuator-Controller-Board-rescue-Attenuator-Controller-Board-rescue BZ1
+L Attenuator-Controller-Board-rescue:CPT-2016-75-SMT-TR-Custom_parts-Attenuator-Controller-Board-rescue-Attenuator-Controller-Board-rescue-Attenuator-Controller-Board-rescue BZ1
 U 1 1 5FE01F50
 P 14450 6900
@@
 $EndComp
 $Comp
-L Mechanical:MountingHole H1
+L Mechanical:MountingHole_Pad H1
 U 1 1 6179BB3F
 P 8700 10250
-F 0 "H1" H 8650 10400 50  0000 L CNN
+F 0 "H1" H 8650 10450 50  0000 L CNN
 F 1 "MountingHole" H 8500 10100 50  0001 L CNN
 F 2 "Custom Footprints:1_4-20_Clearance_hole" H 8700 10250 50  0001 C CNN
@@
 $EndComp
 $Comp
-L Mechanical:MountingHole H2
+L Mechanical:MountingHole_Pad H2
 U 1 1 62040EAE
 P 8850 10250
-F 0 "H2" H 8800 10400 50  0000 L CNN
+F 0 "H2" H 8800 10450 50  0000 L CNN
 F 1 "MountingHole" H 8650 10100 50  0001 L CNN
 F 2 "Custom Footprints:1_4-20_Clearance_hole" H 8850 10250 50  0001 C CNN
@@
 $EndComp
 $Comp
-L Mechanical:MountingHole H3
+L Mechanical:MountingHole_Pad H3
 U 1 1 62049E72
 P 9000 10250
-F 0 "H3" H 8950 10400 50  0000 L CNN
+F 0 "H3" H 8950 10450 50  0000 L CNN
 F 1 "MountingHole" H 8800 10100 50  0001 L CNN
 F 2 "Custom Footprints:1_4-20_Clearance_hole" H 9000 10250 50  0001 C CNN
@@
 $EndComp
 $Comp
-L Mechanical:MountingHole H4
+L Mechanical:MountingHole_Pad H4
 U 1 1 6204A1A9
 P 9150 10250
-F 0 "H4" H 9100 10400 50  0000 L CNN
+F 0 "H4" H 9100 10450 50  0000 L CNN
 F 1 "MountingHole" H 8950 10100 50  0001 L CNN
 F 2 "Custom Footprints:1_4-20_Clearance_hole" H 9150 10250 50  0001 C CNN
@@
 Wire Wire Line
 	10650 6750 10650 7000
+$Comp
+L power:GND #PWR0101
+U 1 1 61EF3BA8
+P 12650 7700
+F 0 "#PWR0101" H 12650 7450 50  0001 C CNN
+F 1 "GND" H 12655 7527 50  0000 C CNN
+F 2 "" H 12650 7700 50  0001 C CNN
+F 3 "" H 12650 7700 50  0001 C CNN
+	1    12650 7700
+	1    0    0    -1
+$EndComp
+$Comp
+L power:GND #PWR0102
+U 1 1 61EF4408
+P 12650 9050
+F 0 "#PWR0102" H 12650 8800 50  0001 C CNN
+F 1 "GND" H 12655 8877 50  0000 C CNN
+F 2 "" H 12650 9050 50  0001 C CNN
+F 3 "" H 12650 9050 50  0001 C CNN
+	1    12650 9050
+	1    0    0    -1
+$EndComp
+$Comp
+L power:GND #PWR0103
+U 1 1 61EF4BA2
+P 13850 9050
+F 0 "#PWR0103" H 13850 8800 50  0001 C CNN
+F 1 "GND" H 13855 8877 50  0000 C CNN
+F 2 "" H 13850 9050 50  0001 C CNN
+F 3 "" H 13850 9050 50  0001 C CNN
+	1    13850 9050
+	1    0    0    -1
+$EndComp
+$Comp
+L power:GND #PWR0104
+U 1 1 61EF5165
+P 15050 9050
+F 0 "#PWR0104" H 15050 8800 50  0001 C CNN
+F 1 "GND" H 15055 8877 50  0000 C CNN
+F 2 "" H 15050 9050 50  0001 C CNN
+F 3 "" H 15050 9050 50  0001 C CNN
+	1    15050 9050
+	1    0    0    -1
+$EndComp
+Wire Wire Line
+	8700 10350 8850 10350
+Connection ~ 8850 10350
+Wire Wire Line
+	8850 10350 9000 10350
+Connection ~ 9000 10350
+Wire Wire Line
+	9000 10350 9150 10350
+$Comp
+L power:GND #PWR?
+U 1 1 61F00536
+P 9150 10350
+F 0 "#PWR?" H 9150 10100 50  0001 C CNN
+F 1 "GND" H 9155 10177 50  0000 C CNN
+F 2 "" H 9150 10350 50  0001 C CNN
+F 3 "" H 9150 10350 50  0001 C CNN
+	1    9150 10350
+	1    0    0    -1
+$EndComp
+Connection ~ 9150 10350
+$Comp
+L power:GND #PWR?
+U 1 1 61F011DF
+P 8700 10350
+F 0 "#PWR?" H 8700 10100 50  0001 C CNN
+F 1 "GND" H 8705 10177 50  0000 C CNN
+F 2 "" H 8700 10350 50  0001 C CNN
+F 3 "" H 8700 10350 50  0001 C CNN
+	1    8700 10350
+	1    0    0    -1
+$EndComp
+Connection ~ 8700 10350
 $EndSCHEMATC

Commit message: Optional grounding of standoffs - ordered revision
Parts:
- added JP1, JP2, JP3, JP4: Jumper_NC_Small, Jumper:SolderJumper-2_P1.3mm_Open_TrianglePad1.0x1.5mm, symbol Device:Jumper_NO_Small
- BZ1: symbol Attenuator-Controller-Board-rescue:CPT-2016-75-SMT-TR-Custom_parts-Attenuator-Controller-Board-rescue-Attenuator-Controller-Board-rescue-Attenuator-Controller-Board-rescue -> Attenuator-Controller-Board-rescue:CPT-2016-75-SMT-TR-Custom_parts-Attenuator-Controller-Board-rescue-Attenuator-Controller-Board-rescue-Attenuator-Controller-Board-rescue-Attenuator-Controller-Board-rescue
- D1: symbol Attenuator-Controller-Board-rescue:BAT54BRW-Custom_parts-Attenuator-Controller-Board-rescue-Attenuator-Controller-Board-rescue-Attenuator-Controller-Board-rescue -> Attenuator-Controller-Board-rescue:BAT54BRW-Custom_parts-Attenuator-Controller-Board-rescue-Attenuator-Controller-Board-rescue-Attenuator-Controller-Board-rescue-Attenuator-Controller-Board-rescue
- renumbered H3 to H1, H4 to H2, H1 to H3, H2 to H4
Connections:
- net GND: now also JP1.2, JP2.2, JP3.2, JP4.2; no longer H1.1, H2.1, H3.1, H4.1
- new net: H3.1, JP3.1
- new net: H4.1, JP4.1
- new net: H1.1, JP1.1
- new net: H2.1, JP2.1
Other:
- moved on the sheet: H1, H2, H3, H4
Changed lines of the file:
@@
 	13800 3000 14550 3000
 $Comp
-L Attenuator-Controller-Board-rescue:BAT54BRW-Custom_parts-Attenuator-Controller-Board-rescue-Attenuator-Controller-Board-rescue-Attenuator-Controller-Board-rescue D1
+L Attenuator-Controller-Board-rescue:BAT54BRW-Custom_parts-Attenuator-Controller-Board-rescue-Attenuator-Controller-Board-rescue-Attenuator-Controller-Board-rescue-Attenuator-Controller-Board-rescue D1
 U 1 1 5F7E5C45
 P 8850 5300
@@
 Audible alarm
 $Comp
-L Attenuator-Controller-Board-rescue:CPT-2016-75-SMT-TR-Custom_parts-Attenuator-Controller-Board-rescue-Attenuator-Controller-Board-rescue-Attenuator-Controller-Board-rescue BZ1
+L Attenuator-Controller-Board-rescue:CPT-2016-75-SMT-TR-Custom_parts-Attenuator-Controller-Board-rescue-Attenuator-Controller-Board-rescue-Attenuator-Controller-Board-rescue-Attenuator-Controller-Board-rescue BZ1
 U 1 1 5FE01F50
 P 14450 6900
@@
 $EndComp
 $Comp
+L Mechanical:MountingHole_Pad H3
+U 1 1 6179BB3F
+P 9150 9950
+F 0 "H3" H 9100 10150 50  0000 L CNN
+F 1 "MountingHole" H 8950 9800 50  0001 L CNN
+F 2 "Custom Footprints:1_4-20_Clearance_hole" H 9150 9950 50  0001 C CNN
+F 3 "http://dpk3n3gg92jwt.cloudfront.net/domains/raf/pdf/RAF%20Catalog.pdf" H 9150 9950 50  0001 C CNN
+F 4 "RAF Electronic Hardware" H 9150 9950 50  0001 C CNN "Manufacturer"
+F 5 "4689-2520-S-12" H 9150 9950 50  0001 C CNN "Part #"
+	1    9150 9950
+	1    0    0    -1
+$EndComp
+$Comp
+L Mechanical:MountingHole_Pad H4
+U 1 1 62040EAE
+P 9400 9950
+F 0 "H4" H 9350 10150 50  0000 L CNN
+F 1 "MountingHole" H 9200 9800 50  0001 L CNN
+F 2 "Custom Footprints:1_4-20_Clearance_hole" H 9400 9950 50  0001 C CNN
+F 3 "http://dpk3n3gg92jwt.cloudfront.net/domains/raf/pdf/RAF%20Catalog.pdf" H 9400 9950 50  0001 C CNN
+F 4 "RAF Electronic Hardware" H 9400 9950 50  0001 C CNN "Manufacturer"
+F 5 "4689-2520-S-12" H 9400 9950 50  0001 C CNN "Part #"
+	1    9400 9950
+	1    0    0    -1
+$EndComp
+$Comp
 L Mechanical:MountingHole_Pad H1
-U 1 1 6179BB3F
-P 8700 10250
-F 0 "H1" H 8650 10450 50  0000 L CNN
-F 1 "MountingHole" H 8500 10100 50  0001 L CNN
-F 2 "Custom Footprints:1_4-20_Clearance_hole" H 8700 10250 50  0001 C CNN
-F 3 "http://dpk3n3gg92jwt.cloudfront.net/domains/raf/pdf/RAF%20Catalog.pdf" H 8700 10250 50  0001 C CNN
-F 4 "RAF Electronic Hardware" H 8700 10250 50  0001 C CNN "Manufacturer"
-F 5 "4689-2520-S-12" H 8700 10250 50  0001 C CNN "Part #"
-	1    8700 10250
+U 1 1 62049E72
+P 8650 9950
+F 0 "H1" H 8600 10150 50  0000 L CNN
+F 1 "MountingHole" H 8450 9800 50  0001 L CNN
+F 2 "Custom Footprints:1_4-20_Clearance_hole" H 8650 9950 50  0001 C CNN
+F 3 "http://dpk3n3gg92jwt.cloudfront.net/domains/raf/pdf/RAF%20Catalog.pdf" H 8650 9950 50  0001 C CNN
+F 4 "RAF Electronic Hardware" H 8650 9950 50  0001 C CNN "Manufacturer"
+F 5 "4689-2520-S-12" H 8650 9950 50  0001 C CNN "Part #"
+	1    8650 9950
 	1    0    0    -1
 $EndComp
 $Comp
 L Mechanical:MountingHole_Pad H2
-U 1 1 62040EAE
-P 8850 10250
-F 0 "H2" H 8800 10450 50  0000 L CNN
-F 1 "MountingHole" H 8650 10100 50  0001 L CNN
-F 2 "Custom Footprints:1_4-20_Clearance_hole" H 8850 10250 50  0001 C CNN
-F 3 "http://dpk3n3gg92jwt.cloudfront.net/domains/raf/pdf/RAF%20Catalog.pdf" H 8850 10250 50  0001 C CNN
-F 4 "RAF Electronic Hardware" H 8850 10250 50  0001 C CNN "Manufacturer"
-F 5 "4689-2520-S-12" H 8850 10250 50  0001 C CNN "Part #"
-	1    8850 10250
-	1    0    0    -1
-$EndComp
-$Comp
-L Mechanical:MountingHole_Pad H3
-U 1 1 62049E72
-P 9000 10250
-F 0 "H3" H 8950 10450 50  0000 L CNN
-F 1 "MountingHole" H 8800 10100 50  0001 L CNN
-F 2 "Custom Footprints:1_4-20_Clearance_hole" H 9000 10250 50  0001 C CNN
-F 3 "http://dpk3n3gg92jwt.cloudfront.net/domains/raf/pdf/RAF%20Catalog.pdf" H 9000 10250 50  0001 C CNN
-F 4 "RAF Electronic Hardware" H 9000 10250 50  0001 C CNN "Manufacturer"
-F 5 "4689-2520-S-12" H 9000 10250 50  0001 C CNN "Part #"
-	1    9000 10250
-	1    0    0    -1
-$EndComp
-$Comp
-L Mechanical:MountingHole_Pad H4
 U 1 1 6204A1A9
-P 9150 10250
-F 0 "H4" H 9100 10450 50  0000 L CNN
-F 1 "MountingHole" H 8950 10100 50  0001 L CNN
-F 2 "Custom Footprints:1_4-20_Clearance_hole" H 9150 10250 50  0001 C CNN
-F 3 "http://dpk3n3gg92jwt.cloudfront.net/domains/raf/pdf/RAF%20Catalog.pdf" H 9150 10250 50  0001 C CNN
-F 4 "RAF Electronic Hardware" H 9150 10250 50  0001 C CNN "Manufacturer"
-F 5 "4689-2520-S-12" H 9150 10250 50  0001 C CNN "Part #"
-	1    9150 10250
+P 8900 9950
+F 0 "H2" H 8850 10150 50  0000 L CNN
+F 1 "MountingHole" H 8700 9800 50  0001 L CNN
+F 2 "Custom Footprints:1_4-20_Clearance_hole" H 8900 9950 50  0001 C CNN
+F 3 "http://dpk3n3gg92jwt.cloudfront.net/domains/raf/pdf/RAF%20Catalog.pdf" H 8900 9950 50  0001 C CNN
+F 4 "RAF Electronic Hardware" H 8900 9950 50  0001 C CNN "Manufacturer"
+F 5 "4689-2520-S-12" H 8900 9950 50  0001 C CNN "Part #"
+	1    8900 9950
 	1    0    0    -1
 $EndComp
@@
 	1    0    0    -1
 $EndComp
-Wire Wire Line
-	8700 10350 8850 10350
-Connection ~ 8850 10350
-Wire Wire Line
-	8850 10350 9000 10350
-Connection ~ 9000 10350
-Wire Wire Line
-	9000 10350 9150 10350
-$Comp
-L power:GND #PWR?
-U 1 1 61F00536
-P 9150 10350
-F 0 "#PWR?" H 9150 10100 50  0001 C CNN
-F 1 "GND" H 9155 10177 50  0000 C CNN
-F 2 "" H 9150 10350 50  0001 C CNN
-F 3 "" H 9150 10350 50  0001 C CNN
-	1    9150 10350
-	1    0    0    -1
-$EndComp
-Connection ~ 9150 10350
-$Comp
-L power:GND #PWR?
-U 1 1 61F011DF
-P 8700 10350
-F 0 "#PWR?" H 8700 10100 50  0001 C CNN
-F 1 "GND" H 8705 10177 50  0000 C CNN
-F 2 "" H 8700 10350 50  0001 C CNN
-F 3 "" H 8700 10350 50  0001 C CNN
-	1    8700 10350
-	1    0    0    -1
-$EndComp
-Connection ~ 8700 10350
+$Comp
+L Device:Jumper_NO_Small JP3
+U 1 1 61F08E3C
+P 9150 10150
+F 0 "JP3" V 9150 10200 50  0000 L CNN
+F 1 "Jumper_NC_Small" V 9195 10198 50  0001 L CNN
+F 2 "Jumper:SolderJumper-2_P1.3mm_Open_TrianglePad1.0x1.5mm" H 9150 10150 50  0001 C CNN
+F 3 "~" H 9150 10150 50  0001 C CNN
+	1    9150 10150
+	0    1    1    0
+$EndComp
+$Comp
+L Device:Jumper_NO_Small JP4
+U 1 1 61F0B9AC
+P 9400 10150
+F 0 "JP4" V 9400 10200 50  0000 L CNN
+F 1 "Jumper_NC_Small" V 9445 10198 50  0001 L CNN
+F 2 "Jumper:SolderJumper-2_P1.3mm_Open_TrianglePad1.0x1.5mm" H 9400 10150 50  0001 C CNN
+F 3 "~" H 9400 10150 50  0001 C CNN
+	1    9400 10150
+	0    1    1    0
+$EndComp
+$Comp
+L Device:Jumper_NO_Small JP1
+U 1 1 61F0BF25
+P 8650 10150
+F 0 "JP1" V 8650 10200 50  0000 L CNN
+F 1 "Jumper_NC_Small" V 8695 10198 50  0001 L CNN
+F 2 "Jumper:SolderJumper-2_P1.3mm_Open_TrianglePad1.0x1.5mm" H 8650 10150 50  0001 C CNN
+F 3 "~" H 8650 10150 50  0001 C CNN
+	1    8650 10150
+	0    1    1    0
+$EndComp
+$Comp
+L Device:Jumper_NO_Small JP2
+U 1 1 61F0C3FB
+P 8900 10150
+F 0 "JP2" V 8900 10200 50  0000 L CNN
+F 1 "Jumper_NC_Small" V 8945 10198 50  0001 L CNN
+F 2 "Jumper:SolderJumper-2_P1.3mm_Open_TrianglePad1.0x1.5mm" H 8900 10150 50  0001 C CNN
+F 3 "~" H 8900 10150 50  0001 C CNN
+	1    8900 10150
+	0    1    1    0
+$EndComp
+$Comp
+L power:GND #PWR0105
+U 1 1 61F0C867
+P 9150 10250
+F 0 "#PWR0105" H 9150 10000 50  0001 C CNN
+F 1 "GND" H 9155 10077 50  0000 C CNN
+F 2 "" H 9150 10250 50  0001 C CNN
+F 3 "" H 9150 10250 50  0001 C CNN
+	1    9150 10250
+	1    0    0    -1
+$EndComp
+$Comp
+L power:GND #PWR0106
+U 1 1 61F1B3F1
+P 9400 10250
+F 0 "#PWR0106" H 9400 10000 50  0001 C CNN
+F 1 "GND" H 9405 10077 50  0000 C CNN
+F 2 "" H 9400 10250 50  0001 C CNN
+F 3 "" H 9400 10250 50  0001 C CNN
+	1    9400 10250
+	1    0    0    -1
+$EndComp
+$Comp
+L power:GND #PWR0107
+U 1 1 61F1B7A2
+P 8650 10250
+F 0 "#PWR0107" H 8650 10000 50  0001 C CNN
+F 1 "GND" H 8655 10077 50  0000 C CNN
+F 2 "" H 8650 10250 50  0001 C CNN
+F 3 "" H 8650 10250 50  0001 C CNN
+	1    8650 10250
+	1    0    0    -1
+$EndComp
+$Comp
+L power:GND #PWR0108
+U 1 1 61F1BB0A
+P 8900 10250
+F 0 "#PWR0108" H 8900 10000 50  0001 C CNN
+F 1 "GND" H 8905 10077 50  0000 C CNN
+F 2 "" H 8900 10250 50  0001 C CNN
+F 3 "" H 8900 10250 50  0001 C CNN
+	1    8900 10250
+	1    0    0    -1
+$EndComp
 $EndSCHEMATC
